File: BH_Pzem_WI_FI_SHIELD/PzemBoard.brd (EAGLE design)
At the start: 34.3 x 78 mm, 23 parts, among them J6 8p, J7 8p, U1 DS18B20, U2 esp12

Commit message: pista em falta para o GND
Connections:
- removed net N$2: OK1.3
- net GND: now also OK1.3
Routing:
- net GPIO14: track 49.0 -> 14.8 mm
- net GND: track 143.6 -> 157.9 mm
Changed lines of the file:
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@@
 <wire x1="20.51308125" y1="60.706" x2="20.409625" y2="60.80945625" width="0.4064" layer="1"/>
 <contactref element="U1" pad="1"/>
-<wire x1="23.942065625" y1="32.90963125" x2="23.942065625" y2="19.4904" width="0.254" layer="1"/>
+<wire x1="23.942065625" y1="32.90963125" x2="23.942065625" y2="27.686" width="0.254" layer="1"/>
+<wire x1="23.942065625" y1="27.686" x2="23.942065625" y2="19.4904" width="0.254" layer="1"/>
 <wire x1="23.942065625" y1="19.4904" x2="29.69316875" y2="13.739296875" width="0.254" layer="1"/>
 <wire x1="23.942065625" y1="32.90963125" x2="27.876240625" y2="32.90963125" width="0.254" layer="1"/>
@@
 <wire x1="24.892" y1="66.548" x2="24.892" y2="66.294" width="0.254" layer="1"/>
 <wire x1="24.892" y1="66.294" x2="23.114" y2="64.516" width="0.254" layer="1"/>
+<contactref element="OK1" pad="3"/>
+<wire x1="23.942065625" y1="27.686" x2="17.526" y2="27.686" width="0.2" layer="1"/>
+<wire x1="17.526" y1="27.686" x2="11.938" y2="33.274" width="0.2" layer="1"/>
 </signal>
 <signal name="VCC">
@@
 <wire x1="11.938" y1="35.814" x2="12.026" y2="35.902" width="0.254" layer="1"/>
 <wire x1="12.026" y1="35.902" x2="15.24" y2="35.902" width="0.254" layer="1"/>
-<wire x1="17.414990625" y1="44.132090625" x2="18.425015625" y2="44.132090625" width="0.254" layer="16"/>
-<wire x1="18.425015625" y1="44.132090625" x2="19.139209375" y2="43.417896875" width="0.254" layer="16"/>
-<wire x1="21.780796875" y1="43.417896875" x2="22.494990625" y2="44.132090625" width="0.254" layer="16"/>
-<wire x1="29.712509375" y1="42.236228125" x2="29.811146875" y2="42.180178125" width="0.254" layer="16"/>
-<wire x1="29.811146875" y1="42.180178125" x2="29.827325" y2="42.1214125" width="0.254" layer="16"/>
-<wire x1="29.902778125" y1="38.63918125" x2="29.8704" y2="38.542046875" width="0.254" layer="16"/>
-<wire x1="29.900515625" y1="38.64370625" x2="29.902778125" y2="38.63918125" width="0.254" layer="16"/>
-<wire x1="12.769221875" y1="36.645221875" x2="11.938" y2="35.814" width="0.254" layer="16"/>
-<wire x1="22.494990625" y1="44.132090625" x2="26.970853125" y2="44.132090625" width="0.254" layer="16"/>
-<wire x1="26.970853125" y1="44.132090625" x2="27.67335" y2="43.42959375" width="0.254" layer="16"/>
-<wire x1="27.67335" y1="43.42959375" x2="27.867453125" y2="43.31929375" width="0.254" layer="16"/>
-<wire x1="15.38" y1="42.912884375" x2="16.195784375" y2="42.912884375" width="0.254" layer="16"/>
-<wire x1="16.195784375" y1="42.912884375" x2="17.414990625" y2="44.132090625" width="0.254" layer="16"/>
-<wire x1="27.867453125" y1="43.31929375" x2="28.62944375" y2="43.31929375" width="0.254" layer="16"/>
-<wire x1="28.62944375" y1="43.31929375" x2="29.712509375" y2="42.236228125" width="0.254" layer="16"/>
-<wire x1="29.827325" y1="42.1214125" x2="29.900515625" y2="42.048221875" width="0.254" layer="16"/>
-<wire x1="29.8704" y1="38.542046875" x2="29.8704" y2="38.393875" width="0.254" layer="16"/>
-<wire x1="29.900515625" y1="42.048221875" x2="29.900515625" y2="38.64370625" width="0.254" layer="16"/>
-<wire x1="29.8704" y1="38.393875" x2="28.121746875" y2="36.645221875" width="0.254" layer="16"/>
-<wire x1="28.121746875" y1="36.645221875" x2="12.769221875" y2="36.645221875" width="0.254" layer="16"/>
-<wire x1="21.780796875" y1="41.275590625" x2="21.780796875" y2="43.417896875" width="0.254" layer="16"/>
-<wire x1="19.139209375" y1="43.417896875" x2="19.139209375" y2="42.437196875" width="0.254" layer="16"/>
-<wire x1="19.139209375" y1="42.437196875" x2="20.300815625" y2="41.275590625" width="0.254" layer="16"/>
-<wire x1="20.300815625" y1="41.275590625" x2="21.780796875" y2="41.275590625" width="0.254" layer="16"/>
+<wire x1="11.938" y1="35.814" x2="11.938" y2="38.608" width="0.2" layer="16"/>
+<wire x1="15.38" y1="42.05" x2="15.38" y2="42.912884375" width="0.2" layer="16"/>
+<wire x1="11.938" y1="38.608" x2="15.38" y2="42.05" width="0.2" layer="16"/>
 </signal>
 <signal name="GPIO16">
@@
 <wire x1="0.254" y1="35.394" x2="0" y2="35.14" width="0.254" layer="1"/>
 </signal>
-<signal name="N$2">
-<contactref element="OK1" pad="3"/>
-</signal>
 <signal name="SIGNAL_GND">
