File: BH_Pzem_WI_FI_SHIELD_rev_1.1/BH_Pzem_WI_FI_SHIELD_rev_1.1.brd (EAGLE design)
At the start: 34.3 x 78 mm, 23 parts, among them J6 8p, J7 8p, U1 DS18B20, U2 esp12

Commit message: Código melhorado, Board rev1.1 in progress
Parts:
- moved U$2 0.39 mm to (15.2, 21.7), flipped to the top, turned to 0 degrees
Connections:
- removed net VCC_D: J1.1, J6.9
- net GPIO04: now also J1.3, J6.5; no longer J1.2, J6.6
- net GPIO05: now also J1.2, J6.6; no longer J1.3, J6.5
- net VCC: now also J1.1, J6.9
Routing:
- net 3V3: track 123.4 -> 31.3 mm, vias 1 -> 0
- net GND: track 157.9 -> 69.3 mm
- net GPIO12: track 73.0 -> 14.6 mm
- net FASE_IN: track 30.0 -> 5.11 mm
- net CH_PD: track 25.8 -> 2.56 mm, vias 1 -> 0
- net GPIO0: track 25.7 -> 4.37 mm
- net GPIO15: track 15.9 -> 3.29 mm, vias 1 -> 0
- net NEUTRAL_IN_FUSED: track 9.72 -> 0.00 mm
- net VCC_D: track 9.50 -> 0.00 mm
- net VCC: track 31.5 -> 38.8 mm, vias 1 -> 0
Other:
- outline, holes or cut-outs redrawn
- board text added: "L"
- board text removed: "F"

Commit message: rev 1.1 board
Parts:
- moved R11 14.4 mm to (21.6, 67.6), turned to 90 degrees
- moved R10 14.1 mm to (29.8, 63.9), turned to 90 degrees
- moved R3 4.33 mm to (30.5, 36.8)
- moved R8 3.77 mm to (28.0, 53.4), turned to 270 degrees
- moved R9 2.96 mm to (25.5, 53.2), turned to 270 degrees
- moved FLASH 2.71 mm to (27.9, 58.5), turned to 90 degrees
- moved U1 2.03 mm to (25.5, 66.0), turned to 300 degrees
- moved RESET 0.76 mm to (27.7, 46.2), turned to 270 degrees
- moved F1 0.51 mm to (2.91, 9.40)
Connections:
- net NEUTRAL_IN renamed NEUTRAL
- removed net FASE_IN: U$1.P$2, U$2.P$2, X3.2
- removed net NEUTRAL_IN_FUSED: F1.P$2, U$2.P$1
- new net LINE: U$1.P$2, U$2.P$1, X3.2
- new net NEUTRAL_FUSED: F1.P$2, U$2.P$2
Routing:
- net VCC: track 38.8 -> 100.3 mm, vias 0 -> 1
- net GPIO12: track 14.6 -> 50.2 mm
- net LINE: track 0.00 -> 31.8 mm
- net 3V3: track 31.3 -> 60.6 mm
- net GND: track 69.3 -> 90.5 mm, vias 1 -> 3
- net CH_PD: track 2.56 -> 23.6 mm
- net GPIO0: track 4.37 -> 21.3 mm
- net NEUTRAL_FUSED: track 0.00 -> 9.87 mm
- net FASE_IN: track 5.11 -> 0.00 mm
- net GPIO15: track 3.29 -> 7.27 mm
- net RESET: track 42.1 -> 43.4 mm, vias 0 -> 1
Other:
- outline, holes or cut-outs redrawn
