File: pcb_rev_1_2/BH_Pzem_WI_FI_SHIELD.brd (EAGLE design)
At the start: 34.3 x 78 mm, 23 parts, among them J6 8p, J7 8p, U1 DS18B20, U2 esp12

Commit message: PCB REV 1.2. Melhorias - Pistas de alimentação mais largas - Orifícios de header 250v mais largos - Adicionado um header para extender o numero de sensores de temperatura (DS18b28_ext)
Parts:
- added DS18B28_EXT: (no value), SparkFun-Connectors:1X03
Connections:
- net 3V3: now also DS18B28_EXT.1
- net GND: now also DS18B28_EXT.3
- net GPIO12: now also DS18B28_EXT.2
Routing:
- net 3V3: track 60.6 -> 80.1 mm
- net GND: track 90.5 -> 108.1 mm
- net GPIO12: track 50.2 -> 67.4 mm
- net VCC: track 100.3 -> 103.1 mm
- net CH_PD: track 23.6 -> 26.0 mm
- net GPIO0: track 21.3 -> 22.7 mm
Other:
- board text added: "rev1.2"
- board text removed: "rev1.1"
