File: pcb_rev_1_2/BH_Pzem_WI_FI_SHIELD.sch (EAGLE design)
At the start: 23 parts, among them J6 8p, J7 8p, U1 DS18B20, U2 esp12

Commit message: PCB REV 1.2. Melhorias - Pistas de alimentação mais largas - Orifícios de header 250v mais largos - Adicionado um header para extender o numero de sensores de temperatura (DS18b28_ext)
Parts:
- added DS18B28_EXT: (no value), SparkFun-Connectors:CONN_03
Connections:
- net 3V3: now also DS18B28_EXT.1
- net GND: now also DS18B28_EXT.3
- net GPIO12: now also DS18B28_EXT.2
Changed lines of the file:
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@@
 <part name="U$1" library="captain-slow" deviceset="SCREWTERMINALS_5MM_2" device=""/>
 <part name="J3" library="SparkFun-Connectors" library_urn="urn:adsk.eagle:library:513" deviceset="CONN_02" device="" package3d_urn="urn:adsk.eagle:package:38039/1"/>
+<part name="DS18B28_EXT" library="SparkFun-Connectors" library_urn="urn:adsk.eagle:library:513" deviceset="CONN_03" device="" package3d_urn="urn:adsk.eagle:package:38063/1"/>
 </parts>
 <sheets>
@@
 <instance part="U$1" gate="G$1" x="124.46" y="43.18"/>
 <instance part="J3" gate="G$1" x="17.78" y="45.72" rot="R270"/>
+<instance part="DS18B28_EXT" gate="J$1" x="254" y="88.9" rot="R180"/>
 </instances>
 <busses>
@@
 <label x="63.5" y="17.78" size="1.778" layer="95" xref="yes"/>
 </segment>
+<segment>
+<pinref part="DS18B28_EXT" gate="J$1" pin="3"/>
+<wire x1="246.38" y1="86.36" x2="241.3" y2="86.36" width="0.1524" layer="91"/>
+<label x="241.3" y="86.36" size="1.778" layer="95" rot="R180" xref="yes"/>
+</segment>
 </net>
 <net name="VCC" class="0">
@@
 <wire x1="187.96" y1="83.82" x2="180.34" y2="83.82" width="0.1524" layer="91"/>
 <label x="180.34" y="83.82" size="1.778" layer="95" rot="R180" xref="yes"/>
+</segment>
+<segment>
+<pinref part="DS18B28_EXT" gate="J$1" pin="2"/>
+<wire x1="246.38" y1="88.9" x2="231.14" y2="88.9" width="0.1524" layer="91"/>
+<label x="231.14" y="88.9" size="1.778" layer="95" rot="R180" xref="yes"/>
 </segment>
 </net>
@@
 <label x="180.34" y="93.98" size="1.778" layer="95" rot="R180" xref="yes"/>
 </segment>
-</net>
+<segment>
+<pinref part="DS18B28_EXT" gate="J$1" pin="1"/>
+<wire x1="246.38" y1="91.44" x2="241.3" y2="91.44" width="0.1524" layer="91"/>
+<label x="241.3" y="91.44" size="1.778" layer="95" rot="R180" xref="yes"/>
+</segment>
+</net>
