File: PCB R2/BH_Pzem_WI_FI_SHIELD.brd (EAGLE design)
At the start: 34.3 x 78 mm, 27 parts, among them J6 8p, J7 8p, U2 esp12

Commit message: rev2
Parts:
- added F1: 1812L010, polyfuse-smd_10:1812L
- added R4: 10k, resistor:R0603
- moved C5 8.89 mm to (2.54, 36.6)
- moved AMS1117 8.89 mm to (4.57, 27.7)
- moved C1 8.89 mm to (6.35, 36.6)
- moved C2 8.89 mm to (6.35, 42.7)
- moved C3 8.89 mm to (2.79, 42.7)
- moved J3 0.80 mm to (32.3, 10.9), turned to 180 degrees
- moved X1 0.80 mm to (19.6, 2.29)
- moved R5 0.57 mm to (19.1, 9.65)
- moved RESET 0.51 mm to (11.5, 76.0)
- moved FLASH 0.25 mm to (22.3, 75.9)
Connections:
- new net N$2: F1.1, X1.2
- net 3V3: now also J1.4, J2.4, J4.4, J5.3, R4.2
- net GND: now also J1.1, J2.1, J4.1, J5.1
- net GPIO04: now also J4.3
- net GPIO05: now also J2.3
- net GPIO12: now also J5.2, R4.1
- net LINE_L: now also F1.2
- net NEUTRAL_IN: now also X1.1
- net RX: now also J1.2, J2.2, J4.2
- net TX: now also J1.3
Routing:
- net NEUTRAL_IN: track 0.00 -> 12.0 mm
- net LINE_L: track 0.00 -> 9.51 mm
- net N$2: track 0.00 -> 6.63 mm
Other:
- board text added: "00"
- board text added: "02"
- board text added: "04"
- board text added: "05"

Commit message: v2
Parts:
- added DISPLAY: (no value), SparkFun-Connectors:JST-4-PTH-VERT
- added RELAY: (no value), SparkFun-Connectors:JST-3-PTH-VERT
- added RESET1: B3U-1000P-2P-SMD, switches:B3U-1000P
- renumbered J1 to PZEM1, J2 to PZEM2, J3 to DS, J4 to PZEM3, J5 to DS18B20
Connections:
- net 3V3: now also DISPLAY.4
- net GND: now also DISPLAY.3, RELAY.1, RESET1.2
- net GPIO02: now also RESET1.1
- net GPIO13: now also RELAY.2
- net GPIO15: now also DISPLAY.2
- net GPIO16: now also DISPLAY.1
- net VCC: now also RELAY.3

Commit message: rev2
Parts:
- removed J6: 8p, SparkFun-Connectors:1X09
- removed J7: 8p, SparkFun-Connectors:1X08
- removed RESET1: B3U-1000P-2P-SMD, switches:B3U-1000P
- added S1: (no value), switch-omron:B3F-10XX
- added UART: (no value), SparkFun-Connectors:JST-4-PTH-VERT
- moved DISPLAY 43.1 mm to (3.30, 32.0), flipped to the bottom, turned to 90 degrees
- moved RESET 33.3 mm to (3.06, 43.8), turned to 90 degrees
- moved FLASH 32.1 mm to (3.06, 50.2), turned to 270 degrees
- moved R11 30.9 mm to (2.51, 39.1), turned to 0 degrees
- moved R2 30.0 mm to (31.0, 31.0), turned to 0 degrees
- moved RELAY 27.9 mm to (3.30, 22.4), flipped to the bottom, turned to 90 degrees
- moved R7 24.2 mm to (8.54, 50.5)
- moved R10 23.7 mm to (6.15, 50.5)
- moved R9 20.1 mm to (12.8, 50.5), turned to 270 degrees
- moved R3 20.0 mm to (10.7, 50.5), turned to 270 degrees
- moved C2 19.6 mm to (25.7, 39.1), turned to 270 degrees
- moved R8 18.0 mm to (22.8, 50.5), turned to 90 degrees
- moved C1 16.6 mm to (22.8, 39.1), turned to 270 degrees
- moved AMS1117 16.4 mm to (17.8, 37.4)
- moved F1 14.3 mm to (25.1, 9.14)
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Connections:
- net 3V3: now also UART.4; no longer J7.1, PZEM1.4, PZEM2.4, PZEM3.4
- net ADC: no longer J7.7
- net CH_PD: no longer J7.6
- net GND: now also S1.1, S1.2, UART.1; no longer J6.1, RESET1.2
- net GPIO0: no longer J6.4
- net GPIO02: now also S1.3, S1.4; no longer J6.3, RESET1.1
- net GPIO04: no longer J6.5
- net GPIO05: no longer J6.6
- net GPIO12: no longer J7.3
- net GPIO13: no longer J7.2
- net GPIO14: no longer J7.4
- net GPIO15: no longer J6.2
- net GPIO16: no longer J7.5
- net RESET: no longer J7.8
- net RX: now also UART.3; no longer J6.7
- net TX: now also UART.2; no longer J6.8
- net VCC: now also PZEM1.4, PZEM2.4, PZEM3.4; no longer J6.9
Routing:
- net GND: track 0.00 -> 183.6 mm, vias 0 -> 4
- net 3V3: track 0.00 -> 155.3 mm, vias 0 -> 2
- net VCC: track 0.00 -> 95.7 mm, vias 0 -> 1
- net GPIO15: track 0.00 -> 60.7 mm, vias 0 -> 1
- net RX: track 0.00 -> 58.4 mm
- net GPIO13: track 0.00 -> 51.9 mm, vias 0 -> 1
- net GPIO0: track 0.00 -> 47.7 mm
- net TX: track 0.00 -> 45.1 mm
- net GPIO14: track 0.00 -> 37.1 mm
- net GPIO04: track 0.00 -> 31.2 mm, vias 0 -> 2
- net GPIO16: track 0.00 -> 30.1 mm
- net GPIO05: track 0.00 -> 25.2 mm
- net GPIO12: track 0.00 -> 25.0 mm
- net RESET: track 0.00 -> 15.0 mm
- net GPIO02: track 0.00 -> 14.7 mm
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- added copper zone on layer 1, net GND
- added copper zone on layer 16, net GND
Other:
- outline, holes or cut-outs redrawn
- board text removed: "00"
- board text removed: "02"
- board text removed: "04"
- board text removed: "05"
- board text removed: "12"
- board text removed: "13"
- board text removed: "14"
- board text removed: "15"
- board text removed: "16"
- board text removed: "3V3"
- board text removed: "ADC"
- board text removed: "EN"
- board text removed: "HLK-PM01"
- board text removed: "RST"
- board text removed: "RX"
- board text removed: "TX"
